File: Luminaries.kicad_sch (KiCad schematic)
At the start: 35 parts, among them J1 12V, J2 ICSP, J3 PGM, J4 CDS, Q1 MMBT3904, Q2 MMBT3904, Q3 MMBT3904, U1 PIC12F683-xSN, U2 AMS1117-5.0

Commit message: updates
Parts:
- renumbered D17 to D12, D12 to D13, D13 to D14, D14 to D15, D15 to D16, D16 to D17, D6 to D2, D5 to D3, D3 to D5, D2 to D6, U2 to U1, U1 to U2
Changed lines of the file:
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@@
 		(dnp no)
 		(fields_autoplaced yes)
-		(property "Reference" "D15"
+		(property "Reference" "D16"
 			(at 240.03 82.8675 90)
 			(show_name no)
@@
 			(project "Luminaries"
 				(path "/57ff6562-df86-4ca6-888d-0cf2b2dca783"
-					(reference "D15")
+					(reference "D16")
 					(unit 1)
 				)
@@
 		(dnp no)
 		(fields_autoplaced yes)
-		(property "Reference" "D6"
+		(property "Reference" "D2"
 			(at 162.56 51.1175 90)
 			(show_name no)
@@
 			(project "Luminaries"
 				(path "/57ff6562-df86-4ca6-888d-0cf2b2dca783"
-					(reference "D6")
+					(reference "D2")
 					(unit 1)
 				)
@@
 		(dnp no)
 		(fields_autoplaced yes)
-		(property "Reference" "#PWR015"
+		(property "Reference" "#PWR018"
 			(at 236.22 129.54 0)
 			(hide yes)
@@
 			(project "Luminaries"
 				(path "/57ff6562-df86-4ca6-888d-0cf2b2dca783"
-					(reference "#PWR015")
+					(reference "#PWR018")
 					(unit 1)
 				)
@@
 		(dnp no)
 		(fields_autoplaced yes)
-		(property "Reference" "U1"
+		(property "Reference" "U2"
 			(at 115.2951 99.06 0)
 			(show_name no)
@@
 			(project "Luminaries"
 				(path "/57ff6562-df86-4ca6-888d-0cf2b2dca783"
-					(reference "U1")
+					(reference "U2")
 					(unit 1)
 				)
@@
 		(in_pos_files yes)
 		(dnp no)
-		(property "Reference" "#PWR017"
+		(property "Reference" "#PWR015"
 			(at 198.12 49.53 0)
 			(hide yes)
@@
 			(project "Luminaries"
 				(path "/57ff6562-df86-4ca6-888d-0cf2b2dca783"
-					(reference "#PWR017")
+					(reference "#PWR015")
 					(unit 1)
 				)
@@
 		(dnp no)
 		(fields_autoplaced yes)
-		(property "Reference" "#PWR010"
+		(property "Reference" "#PWR05"
 			(at 76.2 101.6 0)
 			(hide yes)
@@
 			(project "Luminaries"
 				(path "/57ff6562-df86-4ca6-888d-0cf2b2dca783"
-					(reference "#PWR010")
+					(reference "#PWR05")
 					(unit 1)
 				)
@@
 		(dnp no)
 		(fields_autoplaced yes)
-		(property "Reference" "D16"
+		(property "Reference" "D17"
 			(at 240.03 93.0275 90)
 			(show_name no)
@@
 			(project "Luminaries"
 				(path "/57ff6562-df86-4ca6-888d-0cf2b2dca783"
-					(reference "D16")
+					(reference "D17")
 					(unit 1)
 				)
@@
 		(dnp no)
 		(fields_autoplaced yes)
-		(property "Reference" "#PWR08"
+		(property "Reference" "#PWR012"
 			(at 113.03 143.51 0)
 			(hide yes)
@@
 			(project "Luminaries"
 				(path "/57ff6562-df86-4ca6-888d-0cf2b2dca783"
-					(reference "#PWR08")
+					(reference "#PWR012")
 					(unit 1)
 				)
@@
 		(dnp no)
 		(fields_autoplaced yes)
-		(property "Reference" "#PWR05"
+		(property "Reference" "#PWR03"
 			(at 64.77 64.77 0)
 			(hide yes)
@@
 			(project "Luminaries"
 				(path "/57ff6562-df86-4ca6-888d-0cf2b2dca783"
-					(reference "#PWR05")
+					(reference "#PWR03")
 					(unit 1)
 				)
@@
 		(dnp no)
 		(fields_autoplaced yes)
-		(property "Reference" "#PWR013"
+		(property "Reference" "#PWR014"
 			(at 158.75 129.54 0)
 			(hide yes)
@@
 			(project "Luminaries"
 				(path "/57ff6562-df86-4ca6-888d-0cf2b2dca783"
-					(reference "#PWR013")
+					(reference "#PWR014")
 					(unit 1)
 				)
@@
 		(dnp no)
 		(fields_autoplaced yes)
-		(property "Reference" "D2"
+		(property "Reference" "D6"
 			(at 162.56 91.7575 90)
 			(show_name no)
@@
 			(project "Luminaries"
 				(path "/57ff6562-df86-4ca6-888d-0cf2b2dca783"
-					(reference "D2")
+					(reference "D6")
 					(unit 1)
 				)
@@
 		(dnp no)
 		(fields_autoplaced yes)
-		(property "Reference" "#PWR014"
+		(property "Reference" "#PWR016"
 			(at 198.12 129.54 0)
 			(hide yes)
@@
 			(project "Luminaries"
 				(path "/57ff6562-df86-4ca6-888d-0cf2b2dca783"
-					(reference "#PWR014")
+					(reference "#PWR016")
 					(unit 1)
 				)
@@
 		(dnp no)
 		(fields_autoplaced yes)
-		(property "Reference" "#PWR02"
+		(property "Reference" "#PWR01"
 			(at 46.99 58.42 0)
 			(hide yes)
@@
 			(project "Luminaries"
 				(path "/57ff6562-df86-4ca6-888d-0cf2b2dca783"
-					(reference "#PWR02")
+					(reference "#PWR01")
 					(unit 1)
 				)
@@
 		(in_pos_files yes)
 		(dnp no)
-		(property "Reference" "#PWR011"
+		(property "Reference" "#PWR06"
 			(at 76.2 132.08 0)
 			(hide yes)
@@
 			(project "Luminaries"
 				(path "/57ff6562-df86-4ca6-888d-0cf2b2dca783"
-					(reference "#PWR011")
+					(reference "#PWR06")
 					(unit 1)
 				)
@@
 		(dnp no)
 		(fields_autoplaced yes)
-		(property "Reference" "#PWR04"
+		(property "Reference" "#PWR08"
 			(at 81.28 60.96 0)
 			(hide yes)
@@
 			(project "Luminaries"
 				(path "/57ff6562-df86-4ca6-888d-0cf2b2dca783"
-					(reference "#PWR04")
+					(reference "#PWR08")
 					(unit 1)
 				)
@@
 		(dnp no)
 		(fields_autoplaced yes)
-		(property "Reference" "D3"
+		(property "Reference" "D5"
 			(at 162.56 81.5975 90)
 			(show_name no)
@@
 			(project "Luminaries"
 				(path "/57ff6562-df86-4ca6-888d-0cf2b2dca783"
-					(reference "D3")
+					(reference "D5")
 					(unit 1)
 				)
@@
 		(in_pos_files yes)
 		(dnp no)
-		(property "Reference" "#PWR07"
+		(property "Reference" "#PWR011"
 			(at 113.03 100.33 0)
 			(hide yes)
@@
 			(project "Luminaries"
 				(path "/57ff6562-df86-4ca6-888d-0cf2b2dca783"
-					(reference "#PWR07")
+					(reference "#PWR011")
 					(unit 1)
 				)
@@
 		(in_pos_files yes)
 		(dnp no)
-		(property "Reference" "#PWR03"
+		(property "Reference" "#PWR09"
 			(at 95.25 43.18 0)
 			(hide yes)
@@
 			(project "Luminaries"
 				(path "/57ff6562-df86-4ca6-888d-0cf2b2dca783"
-					(reference "#PWR03")
+					(reference "#PWR09")
 					(unit 1)
 				)
@@
 		(in_pos_files yes)
 		(dnp no)
-		(property "Reference" "#PWR016"
+		(property "Reference" "#PWR013"
 			(at 158.75 48.26 0)
 			(hide yes)
@@
 			(project "Luminaries"
 				(path "/57ff6562-df86-4ca6-888d-0cf2b2dca783"
-					(reference "#PWR016")
+					(reference "#PWR013")
 					(unit 1)
 				)
@@
 		(dnp no)
 		(fields_autoplaced yes)
-		(property "Reference" "D12"
+		(property "Reference" "D13"
 			(at 240.03 52.3875 90)
 			(show_name no)
@@
 			(project "Luminaries"
 				(path "/57ff6562-df86-4ca6-888d-0cf2b2dca783"
-					(reference "D12")
+					(reference "D13")
 					(unit 1)
 				)
@@
 		(dnp no)
 		(fields_autoplaced yes)
-		(property "Reference" "#PWR012"
+		(property "Reference" "#PWR07"
 			(at 76.2 157.48 0)
 			(hide yes)
@@
 			(project "Luminaries"
 				(path "/57ff6562-df86-4ca6-888d-0cf2b2dca783"
-					(reference "#PWR012")
+					(reference "#PWR07")
 					(unit 1)
 				)
@@
 		(in_pos_files yes)
 		(dnp no)
-		(property "Reference" "#PWR01"
+		(property "Reference" "#PWR02"
 			(at 64.77 43.18 0)
 			(hide yes)
@@
 			(project "Luminaries"
 				(path "/57ff6562-df86-4ca6-888d-0cf2b2dca783"
-					(reference "#PWR01")
+					(reference "#PWR02")
 					(unit 1)
 				)
@@
 		(dnp no)
 		(fields_autoplaced yes)
-		(property "Reference" "D14"
+		(property "Reference" "D15"
 			(at 240.03 72.7075 90)
 			(show_name no)
@@
 			(project "Luminaries"
 				(path "/57ff6562-df86-4ca6-888d-0cf2b2dca783"
-					(reference "D14")
+					(reference "D15")
 					(unit 1)
 				)
@@
 		(in_pos_files yes)
 		(dnp no)
-		(property "Reference" "#PWR09"
+		(property "Reference" "#PWR04"
 			(at 76.2 81.28 0)
 			(hide yes)
@@
 			(project "Luminaries"
 				(path "/57ff6562-df86-4ca6-888d-0cf2b2dca783"
-					(reference "#PWR09")
+					(reference "#PWR04")
 					(unit 1)
 				)
@@
 		(dnp no)
 		(fields_autoplaced yes)
-		(property "Reference" "D13"
+		(property "Reference" "D14"
 			(at 240.03 62.5475 90)
 			(show_name no)
@@
 			(project "Luminaries"
 				(path "/57ff6562-df86-4ca6-888d-0cf2b2dca783"
-					(reference "D13")
+					(reference "D14")
 					(unit 1)
 				)
@@
 		(dnp no)
 		(fields_autoplaced yes)
-		(property "Reference" "D17"
+		(property "Reference" "D12"
 			(at 240.03 42.2275 90)
 			(show_name no)
@@
 			(project "Luminaries"
 				(path "/57ff6562-df86-4ca6-888d-0cf2b2dca783"
-					(reference "D17")
+					(reference "D12")
 					(unit 1)
 				)
@@
 		(dnp no)
 		(fields_autoplaced yes)
-		(property "Reference" "D5"
+		(property "Reference" "D3"
 			(at 162.56 61.2775 90)
 			(show_name no)
@@
 			(project "Luminaries"
 				(path "/57ff6562-df86-4ca6-888d-0cf2b2dca783"
-					(reference "D5")
+					(reference "D3")
 					(unit 1)
 				)
@@
 		(in_pos_files yes)
 		(dnp no)
-		(property "Reference" "#PWR018"
+		(property "Reference" "#PWR017"
 			(at 236.22 39.37 0)
 			(hide yes)
@@
 			(project "Luminaries"
 				(path "/57ff6562-df86-4ca6-888d-0cf2b2dca783"
-					(reference "#PWR018")
+					(reference "#PWR017")
 					(unit 1)
 				)
@@
 		(dnp no)
 		(fields_autoplaced yes)
-		(property "Reference" "U2"
+		(property "Reference" "U1"
 			(at 81.28 35.56 0)
 			(show_name no)
@@
 			(project "Luminaries"
 				(path "/57ff6562-df86-4ca6-888d-0cf2b2dca783"
-					(reference "U2")
+					(reference "U1")
 					(unit 1)
 				)
@@
 		(dnp no)
 		(fields_autoplaced yes)
-		(property "Reference" "#PWR06"
+		(property "Reference" "#PWR010"
 			(at 95.25 64.77 0)
 			(hide yes)
@@
 			(project "Luminaries"
 				(path "/57ff6562-df86-4ca6-888d-0cf2b2dca783"
-					(reference "#PWR06")
+					(reference "#PWR010")
 					(unit 1)
 				)

Commit message: Updated pcb.
Parts:
- C1: footprint Package_TO_SOT_SMD:SOT-223-3_TabPin2 -> Capacitor_SMD:CP_Elec_10x10
- C2: footprint Package_TO_SOT_SMD:SOT-223-3_TabPin2 -> Capacitor_SMD:CP_Elec_4x3
- J1: footprint Package_SO:SOIC-8_3.9x4.9mm_P1.27mm -> Connector_BarrelJack:BarrelJack_Horizontal
- J2: footprint (none) -> Connector_PinHeader_2.54mm:PinHeader_1x05_P2.54mm_Vertical
- J3, J4: footprint (none) -> Connector_PinHeader_2.54mm:PinHeader_1x02_P2.54mm_Vertical
- R1, R2, R3, R4, R5, R6, R7: footprint Resistor_THT:R_Array_SIP4 -> Resistor_SMD:R_0805_2012Metric_Pad1.20x1.40mm_HandSolder
Changed lines of the file:
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@@
 			)
 		)
-		(property "Footprint" "Package_SO:SOIC-8_3.9x4.9mm_P1.27mm"
+		(property "Footprint" "Connector_BarrelJack:BarrelJack_Horizontal"
 			(at 38.1 45.466 0)
 			(hide yes)
@@
 			)
 		)
-		(property "Footprint" ""
+		(property "Footprint" "Connector_PinHeader_2.54mm:PinHeader_1x05_P2.54mm_Vertical"
 			(at 68.58 86.36 0)
 			(hide yes)
@@
 			)
 		)
-		(property "Footprint" "Package_TO_SOT_SMD:SOT-223-3_TabPin2"
+		(property "Footprint" "Capacitor_SMD:CP_Elec_10x10"
 			(at 64.77 50.8 0)
 			(hide yes)
@@
 			)
 		)
-		(property "Footprint" "Resistor_THT:R_Array_SIP4"
+		(property "Footprint" "Resistor_SMD:R_0805_2012Metric_Pad1.20x1.40mm_HandSolder"
 			(at 77.216 143.764 90)
 			(hide yes)
@@
 			)
 		)
-		(property "Footprint" "Package_TO_SOT_SMD:SOT-223-3_TabPin2"
+		(property "Footprint" "Capacitor_SMD:CP_Elec_4x3"
 			(at 95.25 50.8 0)
 			(hide yes)
@@
 			)
 		)
-		(property "Footprint" "Resistor_THT:R_Array_SIP4"
+		(property "Footprint" "Resistor_SMD:R_0805_2012Metric_Pad1.20x1.40mm_HandSolder"
 			(at 235.204 101.346 90)
 			(hide yes)
@@
 			)
 		)
-		(property "Footprint" "Resistor_THT:R_Array_SIP4"
+		(property "Footprint" "Resistor_SMD:R_0805_2012Metric_Pad1.20x1.40mm_HandSolder"
 			(at 157.734 101.346 90)
 			(hide yes)
@@
 			)
 		)
-		(property "Footprint" ""
+		(property "Footprint" "Connector_PinHeader_2.54mm:PinHeader_1x02_P2.54mm_Vertical"
 			(at 68.58 116.84 0)
 			(hide yes)
@@
 			)
 		)
-		(property "Footprint" "Resistor_THT:R_Array_SIP4"
+		(property "Footprint" "Resistor_SMD:R_0805_2012Metric_Pad1.20x1.40mm_HandSolder"
 			(at 221.234 113.284 90)
 			(hide yes)
@@
 			)
 		)
-		(property "Footprint" "Resistor_THT:R_Array_SIP4"
+		(property "Footprint" "Resistor_SMD:R_0805_2012Metric_Pad1.20x1.40mm_HandSolder"
 			(at 197.104 101.346 90)
 			(hide yes)
@@
 			)
 		)
-		(property "Footprint" ""
+		(property "Footprint" "Connector_PinHeader_2.54mm:PinHeader_1x02_P2.54mm_Vertical"
 			(at 68.58 135.89 0)
 			(hide yes)
@@
 			)
 		)
-		(property "Footprint" "Resistor_THT:R_Array_SIP4"
+		(property "Footprint" "Resistor_SMD:R_0805_2012Metric_Pad1.20x1.40mm_HandSolder"
 			(at 183.134 113.284 90)
 			(hide yes)
@@
 			)
 		)
-		(property "Footprint" "Resistor_THT:R_Array_SIP4"
+		(property "Footprint" "Resistor_SMD:R_0805_2012Metric_Pad1.20x1.40mm_HandSolder"
 			(at 143.764 113.284 90)
 			(hide yes)
